File: Pico-BLDC-Controller.kicad_sch (KiCad schematic)
At the start: 120 parts, among them J1 Conn_01x02, J2 Conn_01x03, J3 Conn_01x05, J4 SM03B-SRSS-TB, J5 USB_C_Receptacle_USB2.0_14P, J6 Heat Mat, J7 ZJY130-2864KSWLG22, J8 I2C CONN, Q1 SIR680LDP, Q2 SIR680LDP, Q3 SIR680LDP, Q4 SIR680LDP, Q5 SIR680LDP, Q6 SIR680LDP, Q7 DMN3053L-7, SW1 SW_Push, SW2 SW_Push, SW3 RotaryEncoder_Switch, U1 RP2350_60QFN, U10 TPS62822DLC, U2 LMR51430, U3 W25Q128JVS, U4 DRV8350S, U5 WE-TVS-82400102, U6 INA240A2PW, U7 INA240A2PW, U8 INA240A2PW, U9 LMR38020SDDAR, Y1 ABM8-272-T3

Commit message: all
Parts:
- removed C36, C37: 1uF 16V, Capacitor_SMD:C_0603_1608Metric_Pad1.08x0.95mm_HandSolder, symbol MCU_RaspberryPi_RP2350:C
- removed C51, C52: 10uF, Capacitor_SMD:C_0805_2012Metric, symbol MCU_RaspberryPi_RP2350:C
- removed J7: ZJY130-2864KSWLG22, Amphenol_FPC_16:AMPHENOL_F3311A7H121016E200, symbol Amphenol_FPC_16:F3311A7H121016E200
- removed R28: 680k, Resistor_SMD:R_0603_1608Metric_Pad0.98x0.95mm_HandSolder, symbol MCU_RaspberryPi_RP2350:R
- removed R29: 5.1k, Resistor_SMD:R_0603_1608Metric_Pad0.98x0.95mm_HandSolder, symbol MCU_RaspberryPi_RP2350:R
- removed SW3: RotaryEncoder_Switch, Rotary_Encoder:RotaryEncoder_Bourns_Vertical_PEC12R-3x17F-Sxxxx, symbol Device:RotaryEncoder_Switch
- added C20, C21, C31, C51, C59, C68, C71: 100pF, Capacitor_SMD:C_0603_1608Metric_Pad1.08x0.95mm_HandSolder, symbol Device:C
- added C25, C62, C63, C66, C8: 100nF, Capacitor_SMD:C_0603_1608Metric_Pad1.08x0.95mm_HandSolder, symbol MCU_RaspberryPi_RP2350:C
- added C45, C46, C47: C, Capacitor_SMD:C_0603_1608Metric_Pad1.08x0.95mm_HandSolder, symbol Device:C
- added C48, C52, C65: 10pF, Capacitor_SMD:C_0603_1608Metric_Pad1.08x0.95mm_HandSolder, symbol Device:C
- added C49, C50, C64: 100pF, Capacitor_SMD:C_0603_1608Metric_Pad1.08x0.95mm_HandSolder, symbol MCU_RaspberryPi_RP2350:C
- added C57: 4.7uF, Capacitor_SMD:C_0603_1608Metric_Pad1.08x0.95mm_HandSolder, symbol Device:C
- added C58, C72: 0.01uF, Capacitor_SMD:C_0603_1608Metric_Pad1.08x0.95mm_HandSolder, symbol Device:C
- added D3: LED, LED_SMD:LED_0603_1608Metric_Pad1.05x0.95mm_HandSolder, symbol Device:LED
- added J1: Conn_01x10, Connector_JST:JST_PHD_B10B-PHDSS_2x05_P2.00mm_Vertical, symbol Connector_Generic:Conn_01x10
- added R27: 330, Resistor_SMD:R_0603_1608Metric, symbol Device:R
- added R31, R32, R33: R, Resistor_SMD:R_0805_2012Metric_Pad1.20x1.40mm_HandSolder, symbol Device:R
- added TP_1, TP_2, TP_3, TP_GND1: TestPoint, TestPoint:TestPoint_Pad_D1.0mm, symbol Connector:TestPoint
- C1: value 10u -> 100nF; footprint Capacitor_SMD:C_0805_2012Metric -> Capacitor_SMD:C_0603_1608Metric_Pad1.08x0.95mm_HandSolder; MPN DNP -> C0603C104K5RACAUTO; now fitted
- C19: value 10u -> 22uF; footprint Capacitor_SMD:C_0805_2012Metric -> Capacitor_SMD:C_0603_1608Metric_Pad1.08x0.95mm_HandSolder; MPN DNP -> GRM188R60J226MEA0D; now fitted
- C54: renamed from C8; value 100nF -> 100pF; MPN C0603C104K5RACAUTO -> 0603YC101KAT2A
- C61: renamed from C12; value 100nF -> 100pF; MPN C0603C104K5RACAUTO -> 0603YC101KAT2A
- R12: renamed from R24; footprint Resistor_SMD:R_0805_2012Metric -> Resistor_SMD:R_0603_1608Metric; MPN RP0805BRD07100KL -> ERJ-PB3B1003V
- renumbered C50 to C10, C33 to C11, C31 to C12, C41 to C13, C5 to C14, C40 to C15, C42 to C16, C39 to C17, C49 to C18, C27 to C2, C32 to C22, C7 to C23, C4 to C24, C6 to C26, C9 to C27, C10 to C28, C3 to C29, C28 to C3, C44 to C30, C38 to C32, C22 to C33, C48 to C34, C25 to C35, C24 to C36, C43 to C37, C26 to C38, C21 to C39, C34 to C4, C20 to C40, C23 to C41, C47 to C42, C45 to C43, C46 to C44, C29 to C5, C13 to C53, C16 to C55, C14 to C56, C30 to C6, C17 to C60, C11 to C67, C18 to C69, C35 to C7, C15 to C70, C2 to C9, D2 to D1, D1 to D2, J6 to J2, J8 to J3, J5 to J4, J4 to J5, J3 to J6, J1 to J7, J2 to J8, L3 to L1, L4 to L3, L1 to L4, Q7 to Q1, Q3 to Q2, Q5 to Q3, Q6 to Q4, Q4 to Q5, Q2 to Q6, Q1 to Q7, R20 to R1, R1 to R10, R23 to R11, R22 to R13, R25 to R14, R19 to R15, R18 to R16, R11 to R17, R8 to R18, R2 to R19, R21 to R2, R16 to R20, R15 to R21, R17 to R22, R5 to R23, R7 to R24, R31 to R25, R3 to R26, R13 to R28, R14 to R29, R26 to R3, R12 to R30, R27 to R4, R4 to R5, R9 to R6, R10 to R7, R30 to R8, R6 to R9, SW2 to SW1, SW1 to SW2, U2 to U1, U7 to U10, U5 to U2, U9 to U3, U10 to U4, U1 to U5, U3 to U6, U4 to U7, U6 to U9
Connections:
- net +12V: now also TP_2.1
- net +1V1: now also C25.1, C31.1, C59.1, C66.1, C72.1
- net +3V3: now also C20.1, C49.1, C50.1, C51.1, C57.1, C58.1, C62.1, C64.1, C68.1, C71.1, C8.1, D3.2 (A), J1.1 (Pin_1), TP_3.1
- net +5V: now also C21.1, C63.1, TP_1.1
- net CHA_A: now also U5.8 (GPIO5), J1.8 (Pin_8); no longer U5.12 (GPIO8)
- net CHA_B: now also U5.9 (GPIO6), J1.9 (Pin_9); no longer U5.13 (GPIO9)
- net DRV_EN: now also U5.15 (GPIO11); no longer U5.37 (GPIO25)
- net DRV_nFAULT: now also U5.37 (GPIO25), R27.2; no longer U5.15 (GPIO11)
- net GND: now also J6.2 (Pin_2), J7.1 (Pin_1), C20.2, C21.2, C25.2, C31.2, C45.2, C46.2, C47.2, C48.2, C49.2, C50.2, C51.2, C52.2, C57.2, C58.2, C59.2, C62.2, C63.2, C64.2, C65.2, C66.2, C68.2, C71.2, C72.2, C8.2, J1.2 (Pin_2), TP_GND1.1; no longer J6.5 (Pin_5), J7.2 (Pin_2)
- net GPIO0: now also J1.3 (Pin_3)
- net GPIO1: now also J1.4 (Pin_4)
- net GPIO10: now also Q1.1 (G), R2.1
- net GPIO16: now also J6.5 (Pin_5), C48.1; no longer J6.4 (Pin_4)
- net GPIO17: now also J6.4 (Pin_4), C52.1; no longer J6.3 (Pin_3)
- net GPIO18: now also J6.3 (Pin_3), C65.1; no longer J6.2 (Pin_2)
- net GPIO2: now also J1.5 (Pin_5)
- net GPIO26_ADC0: now also U9.8; no longer U8.8
- net GPIO28_ADC2: now also U8.8; no longer U9.8
- net GPIO3: now also J1.6 (Pin_6)
- net GPIO4: now also J1.7 (Pin_7)
- net GPIO7: now also J1.10 (Pin_10); no longer J3.3 (Pin_3), R8.2
- net MOTA_IN: now also R33.1
- net MOTB_IN: now also R32.1
- net MOTC_IN: now also R31.1
- net USB1_D+: now reaches R24.1, U2.1
- net USB1_D-: now reaches R18.1, U2.3
- net at F1.2: now also J7.2 (Pin_2); no longer J7.1 (Pin_1)
- removed net GPIO5: Q1.1 (G), R2.1, U5.8 (GPIO5)
- net GPIO6 renamed GPIO9
- net GPIO9: now also U5.13 (GPIO9); no longer U5.9 (GPIO6)
- new net: D3.1 (K), R27.1
- new net: C47.1, R33.2
- new net: C45.1, R31.2
- new net: C46.1, R32.2
- new net GPIO8: J3.3 (Pin_3), R8.2, U5.12 (GPIO8)
Other:
- note added: "INPUT"
- note added: "ON-CHIP CORE VOLTAGE REGULATOR"
- note added: "OUTPUT"
- note added: "RC Snubber Blank, Value TBA after testing"
- company: (none) -> Manufacturing Future Labs, UCL & Tuah Elektronik 
- title: (none) -> Pico-BLDC-Controller
- moved on the sheet: C10, C13, C14, C15, C16, C17, C18, C9, D1, J4, J6, L3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
