File: Pico-BLDC-Controller.kicad_pcb (KiCad board)
At the start: 4 copper layers, 118 parts, among them J1 Conn_01x02, J2 Conn_01x03, J3 Conn_01x05, J4 SM03B-SRSS-TB, J5 USB_C_Receptacle_USB2.0_14P, J6 Heat Mat, J7 ZJY130-2864KSWLG22, J8 I2C CONN, Q1 SIR680LDP, Q2 SIR680LDP, Q3 SIR680LDP, Q4 SIR680LDP, Q5 SIR680LDP, Q6 SIR680LDP, Q7 DMN3053L-7, SW1 SW_Push, SW2 SW_Push, SW3 RotaryEncoder_Switch, U1 RP2350_60QFN, U10 TPS62822DLC, U2 LMR51430, U3 W25Q128JVS, U4 DRV8350S, U5 WE-TVS-82400102, U6 INA240A2PW, U7 INA240A2PW, U8 INA240A2PW, U9 LMR38020SDDAR, Y1 ABM8-272-T3

Commit message: all
Parts:
- removed the C36 at (50.1, 32.9)
- removed the C37 at (50.1, 35.4)
- removed the J7 at (20.8, 60.8)
- removed the R28 at (67.5, 22.9)
- removed the R29 at (67.5, 25.4)
- removed SW3: RotaryEncoder_Switch, Rotary_Encoder:RotaryEncoder_Bourns_Vertical_PEC12R-3x17F-Sxxxx
- added C1: 100nF, Capacitor_SMD:C_0603_1608Metric_Pad1.08x0.95mm_HandSolder, F.Cu at (113.6, 80.5)
- added C19: 22uF, Capacitor_SMD:C_0603_1608Metric_Pad1.08x0.95mm_HandSolder, F.Cu at (117.3, 67.1)
- added C20: 100pF, Capacitor_SMD:C_0603_1608Metric_Pad1.08x0.95mm_HandSolder, F.Cu at (137.3, 65.3)
- added C21: 100pF, Capacitor_SMD:C_0603_1608Metric_Pad1.08x0.95mm_HandSolder, F.Cu at (115.1, 80.5)
- added C25: 100nF, Capacitor_SMD:C_0603_1608Metric_Pad1.08x0.95mm_HandSolder, F.Cu at (150.2, 53.0)
- added C31: 100pF, Capacitor_SMD:C_0603_1608Metric_Pad1.08x0.95mm_HandSolder, F.Cu at (149.1, 68.4)
- added C45: C, Capacitor_SMD:C_0603_1608Metric_Pad1.08x0.95mm_HandSolder, B.Cu at (183.9, 48.8)
- added C46: C, Capacitor_SMD:C_0603_1608Metric_Pad1.08x0.95mm_HandSolder, B.Cu at (184.0, 63.4)
- added C47: C, Capacitor_SMD:C_0603_1608Metric_Pad1.08x0.95mm_HandSolder, B.Cu at (184.1, 72.0)
- added C48: 10pF, Capacitor_SMD:C_0603_1608Metric_Pad1.08x0.95mm_HandSolder, B.Cu at (158.2, 48.7)
- added C49: 100pF, Capacitor_SMD:C_0603_1608Metric_Pad1.08x0.95mm_HandSolder, B.Cu at (147.2, 53.9)
- added C50: 100pF, Capacitor_SMD:C_0603_1608Metric_Pad1.08x0.95mm_HandSolder, B.Cu at (144.9, 57.6)
- added C57: 4.7uF, Capacitor_SMD:C_0603_1608Metric_Pad1.08x0.95mm_HandSolder, B.Cu at (144.9, 60.6)
- added C58: 0.01uF, Capacitor_SMD:C_0603_1608Metric_Pad1.08x0.95mm_HandSolder, B.Cu at (144.9, 59.1)
- added C59: 100pF, Capacitor_SMD:C_0603_1608Metric_Pad1.08x0.95mm_HandSolder, B.Cu at (156.4, 60.3)
- added C62: 100nF, Capacitor_SMD:C_0603_1608Metric_Pad1.08x0.95mm_HandSolder, B.Cu at (144.9, 62.1)
- added C63: 100nF, Capacitor_SMD:C_0603_1608Metric_Pad1.08x0.95mm_HandSolder, B.Cu at (149.3, 48.1)
- added C64: 100pF, Capacitor_SMD:C_0603_1608Metric_Pad1.08x0.95mm_HandSolder, B.Cu at (151.7, 53.9)
- added C65: 10pF, Capacitor_SMD:C_0603_1608Metric_Pad1.08x0.95mm_HandSolder, B.Cu at (153.1, 48.8)
- added C66: 100nF, Capacitor_SMD:C_0603_1608Metric_Pad1.08x0.95mm_HandSolder, B.Cu at (156.4, 58.8)
- added C68: 100pF, Capacitor_SMD:C_0603_1608Metric_Pad1.08x0.95mm_HandSolder, B.Cu at (147.6, 66.1)
- added C71: 100pF, Capacitor_SMD:C_0603_1608Metric_Pad1.08x0.95mm_HandSolder, B.Cu at (152.0, 66.1)
- added C72: 0.01uF, Capacitor_SMD:C_0603_1608Metric_Pad1.08x0.95mm_HandSolder, B.Cu at (150.5, 66.1)
- added C8: 100nF, Capacitor_SMD:C_0603_1608Metric_Pad1.08x0.95mm_HandSolder, F.Cu at (117.3, 65.6)
- added D3: LED, LED_SMD:LED_0603_1608Metric_Pad1.05x0.95mm_HandSolder, F.Cu at (171.1, 46.5)
- added J1: Conn_01x10, Connector_JST:JST_PHD_B10B-PHDSS_2x05_P2.00mm_Vertical, F.Cu at (98.1, 47.2)
- added R27: 330, Resistor_SMD:R_0603_1608Metric, F.Cu at (171.1, 48.3)
- added R31: R, Resistor_SMD:R_0805_2012Metric_Pad1.20x1.40mm_HandSolder, B.Cu at (183.9, 52.4)
- added R32: R, Resistor_SMD:R_0805_2012Metric_Pad1.20x1.40mm_HandSolder, B.Cu at (184.0, 59.9)
- added R33: R, Resistor_SMD:R_0805_2012Metric_Pad1.20x1.40mm_HandSolder, B.Cu at (184.1, 75.5)
- added TP_1: TestPoint, TestPoint:TestPoint_Pad_D1.0mm, F.Cu at (114.3, 74.8)
- added TP_2: TestPoint, TestPoint:TestPoint_Pad_D1.0mm, F.Cu at (97.0, 74.2)
- added TP_3: TestPoint, TestPoint:TestPoint_Pad_D1.0mm, F.Cu at (115.8, 61.2)
- added TP_GND1: TestPoint, TestPoint:TestPoint_Pad_D1.0mm, F.Cu at (108.0, 63.3)
- C42: renamed from C47; moved to B.Cu
- C43: renamed from C45; moved to B.Cu
- C44: renamed from C46; moved to B.Cu
- C51: value 10uF -> 100pF; footprint Capacitor_SMD:C_0805_2012Metric -> Capacitor_SMD:C_0603_1608Metric_Pad1.08x0.95mm_HandSolder; moved to B.Cu
- C52: value 10uF -> 10pF; footprint Capacitor_SMD:C_0805_2012Metric -> Capacitor_SMD:C_0603_1608Metric_Pad1.08x0.95mm_HandSolder; moved to B.Cu
- C53: renamed from C13; moved to B.Cu
- C54: renamed from C8; value 100nF -> 100pF; moved to B.Cu
- C55: renamed from C16; moved to B.Cu
- C56: renamed from C14; moved to B.Cu
- C60: renamed from C17; moved to B.Cu
- C61: renamed from C12; value 100nF -> 100pF; moved to B.Cu
- C67: renamed from C11; moved to B.Cu
- C69: renamed from C18; moved to B.Cu
- C70: renamed from C15; moved to B.Cu
- R12: renamed from R24; footprint Resistor_SMD:R_0805_2012Metric -> Resistor_SMD:R_0603_1608Metric
- U10: renamed from U7; moved to B.Cu
- U8: moved to B.Cu
- U9: renamed from U6; moved to B.Cu
- moved J7 151.2 mm to (202.6, 84.4), turned to -90 degrees
- moved C37 151.2 mm to (166.2, 85.0), turned to 90 degrees
- moved J5 150.7 mm to (164.3, 45.9), turned to 180 degrees
- moved C43 150.6 mm to (194.0, 79.6), turned to 90 degrees
- moved C44 145.6 mm to (194.0, 67.2), turned to 90 degrees
- moved Q7 144.1 mm to (183.1, 76.5), turned to 180 degrees
- moved C42 142.1 mm to (194.0, 55.0), turned to 90 degrees
- moved Q4 141.6 mm to (182.9, 46.5)
- moved Q6 141.1 mm to (182.9, 69.8)
- moved J8 140.8 mm to (200.2, 65.0), turned to -90 degrees
- moved Q3 139.9 mm to (183.0, 53.2), turned to 180 degrees
- moved Q2 139.4 mm to (183.0, 58.8), turned to 180 degrees
- moved Q5 139.3 mm to (182.9, 64.2)
- moved U7 136.3 mm to (171.1, 59.2), turned to 90 degrees
- moved C40 135.4 mm to (168.5, 68.8), turned to -135 degrees
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- renumbered C50 to C10, C33 to C11, C31 to C12, C41 to C13, C5 to C14, C40 to C15, C42 to C16, C39 to C17, C49 to C18, C27 to C2, C32 to C22, C7 to C23, C4 to C24, C6 to C26, C9 to C27, C10 to C28, C3 to C29, C28 to C3, C44 to C30, C38 to C32, C22 to C33, C48 to C34, C25 to C35, C24 to C36, C43 to C37, C26 to C38, C21 to C39, C34 to C4, C20 to C40, C23 to C41, C29 to C5, C30 to C6, C35 to C7, C2 to C9, D2 to D1, D1 to D2, J6 to J2, J8 to J3, J5 to J4, J4 to J5, J3 to J6, J1 to J7, J2 to J8, L3 to L1, L4 to L3, L1 to L4, Q7 to Q1, Q3 to Q2, Q5 to Q3, Q6 to Q4, Q4 to Q5, Q2 to Q6, Q1 to Q7, R20 to R1, R1 to R10, R23 to R11, R22 to R13, R25 to R14, R19 to R15, R18 to R16, R11 to R17, R8 to R18, R2 to R19, R21 to R2, R16 to R20, R15 to R21, R17 to R22, R5 to R23, R7 to R24, R31 to R25, R3 to R26, R13 to R28, R14 to R29, R26 to R3, R12 to R30, R27 to R4, R4 to R5, R9 to R6, R10 to R7, R30 to R8, R6 to R9, SW2 to SW1, SW1 to SW2, U2 to U1, U5 to U2, U9 to U3, U10 to U4, U1 to U5, U3 to U6, U4 to U7
Connections:
- net Net-(R7-Pad1) renamed /USB1_D+
- net Net-(R8-Pad1) renamed /USB1_D-
- C51 pad 1: Net-(C51-Pad1) -> +3V3
- C52 pad 1: Net-(C52-Pad1) -> /GPIO17
- F1 pad 2: Net-(J1-Pin_1) -> Net-(J7-Pin_2)
- J3 pad 3: /GPIO7 -> /GPIO8
- J3 pad 4: /GPIO6 -> /GPIO9
- J6 pad 2: /GPIO18 -> GND
- J6 pad 3: /GPIO17 -> /GPIO18
- J6 pad 4: /GPIO16 -> /GPIO17
- J6 pad 5: GND -> /GPIO16
- J7 pad 1: Net-(J1-Pin_1) -> GND
- J7 pad 2: GND -> Net-(J7-Pin_2)
- Q1 pad 1: /GPIO5 -> /GPIO10
- R2 pad 1: /GPIO5 -> /GPIO10
- R25 pad 2: /GPIO6 -> /GPIO9
- R8 pad 2: /GPIO7 -> /GPIO8
- U5 pad 12: /CHA_A -> /GPIO8
- U5 pad 13: /CHA_B -> /GPIO9
- U5 pad 15: /DRV_nFAULT -> /DRV_EN
- U5 pad 37: /DRV_EN -> /DRV_nFAULT
- U5 pad 8: /GPIO5 -> /CHA_A
- U5 pad 9: /GPIO6 -> /CHA_B
- U8 pad 8: /GPIO26_ADC0 -> /GPIO28_ADC2
- U9 pad 8: /GPIO28_ADC2 -> /GPIO26_ADC0
Routing:
- net +3V3: track 0.00 -> 191.2 mm, vias 0 -> 49
- net +5V: track 0.00 -> 100.1 mm, vias 0 -> 2
- net /GPIO26_ADC0: track 0.00 -> 85.3 mm, vias 0 -> 1
- net /GPIO27_ADC1: track 0.00 -> 74.6 mm, vias 0 -> 1
- net /GPIO0: track 0.00 -> 70.0 mm, vias 0 -> 1
- net /GPIO4: track 0.00 -> 68.9 mm, vias 0 -> 1
- net /GPIO2: track 0.00 -> 67.7 mm, vias 0 -> 1
- net /CHA_B: track 0.00 -> 67.2 mm, vias 0 -> 1
- net /GPIO1: track 0.00 -> 66.4 mm, vias 0 -> 1
- net /CHA_A: track 0.00 -> 65.6 mm, vias 0 -> 1
- net /GPIO28_ADC2: track 0.00 -> 64.6 mm, vias 0 -> 1
- net /GPIO3: track 0.00 -> 64.0 mm, vias 0 -> 1
- net /GPIO7: track 0.00 -> 63.1 mm, vias 0 -> 1
- net /GPIO10: track 0.00 -> 60.3 mm, vias 0 -> 3
- net /GPIO29_ADC3: track 0.00 -> 58.6 mm, vias 0 -> 2
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- added copper zone on F.Cu, net +12V
- added copper zone on F.Cu, net +1V1
- added copper zone on F.Cu, net +3V3
- added copper zone on In2.Cu, net +3V3
- added copper zone on F.Cu, net +5V
- added copper zone on B.Cu, net /MOTA_IN
- added copper zone on F.Cu, net /MOTA_IN
- added copper zone on In1.Cu, net /MOTA_IN
- added copper zone on In2.Cu, net /MOTA_IN
- added copper zone on B.Cu, net /MOTA_OUT
- added copper zone on F.Cu, net /MOTA_OUT
- added copper zone on In1.Cu, net /MOTA_OUT
- added copper zone on In2.Cu, net /MOTA_OUT
- added copper zone on B.Cu, net /MOTB_IN
- added copper zone on F.Cu, net /MOTB_IN
- added copper zone on In1.Cu, net /MOTB_IN
- added copper zone on In2.Cu, net /MOTB_IN
- added copper zone on B.Cu, net /MOTB_OUT
- added copper zone on F.Cu, net /MOTB_OUT
- added copper zone on In1.Cu, net /MOTB_OUT
- added copper zone on In2.Cu, net /MOTB_OUT
- added copper zone on B.Cu, net /MOTC_IN
- added copper zone on F.Cu, net /MOTC_IN
- added copper zone on In1.Cu, net /MOTC_IN
- added copper zone on In2.Cu, net /MOTC_IN
- added copper zone on B.Cu, net /MOTC_OUT
- added copper zone on F.Cu, net /MOTC_OUT
- added copper zone on In1.Cu, net /MOTC_OUT
- added copper zone on In2.Cu, net /MOTC_OUT
- added copper zone on B.Cu, net GND
- added copper zone on F.Cu, net GND
- added copper zone on In1.Cu, net GND
- added copper zone on In2.Cu, net GND
- added copper zone on B.Cu, net Net-(J7-Pin_2)
- added copper zone on F.Cu, net Net-(J7-Pin_2)
- added copper zone on In1.Cu, net Net-(J7-Pin_2)
- added copper zone on In2.Cu, net Net-(J7-Pin_2)
- added copper zone on B.Cu, net VM
- added copper zone on F.Cu, net VM
- added copper zone on In1.Cu, net VM
- added copper zone on In2.Cu, net VM
Other:
- board outline added: 115 x 55 mm
- board text added: "A"
- board text added: "B"
- board text added: "C"
- board text added: "FAULT"

Commit message: all
Parts:
- added G***: LOGO, Syauqi_logo:SYAUQI, B.Cu at (119.6, 84.5)
- added H1: MountingHole, MountingHole:MountingHole_2.7mm_M2.5_ISO14580, F.Cu at (204.9, 92.6)
- added H2: MountingHole, MountingHole:MountingHole_2.7mm_M2.5_ISO14580, F.Cu at (204.9, 45.6)
- added H3: MountingHole, MountingHole:MountingHole_2.7mm_M2.5_ISO14580, F.Cu at (98.4, 54.1)
- added H4: MountingHole, MountingHole:MountingHole_2.7mm_M2.5_ISO14580, F.Cu at (98.4, 92.6)
- added REF**: ESD-Logo_6.6x6mm_SilkScreen, Symbol:ESD-Logo_6.6x6mm_SilkScreen, F.Cu at (122.2, 59.8)
- added REF**: Symbol_HighVoltage_Triangle_6x6mm_Copper, Symbol:Symbol_HighVoltage_Triangle_6x6mm_Copper, F.Cu at (187.4, 93.5)
- added REF**: Symbol_HighVoltage_Triangle_6x6mm_Copper, Symbol:Symbol_HighVoltage_Triangle_6x6mm_Copper, F.Cu at (191.8, 54.1)
- added REF**: Symbol_HighVoltage_Triangle_6x6mm_Copper, Symbol:Symbol_HighVoltage_Triangle_6x6mm_Copper, F.Cu at (191.7, 67.1)
- added REF**: OSHW-Logo_5.7x6mm_SilkScreen, Symbol:OSHW-Logo_5.7x6mm_SilkScreen, F.Cu at (112.5, 47.8)
- added REF**: OSHW-Logo_5.7x6mm_SilkScreen, Symbol:OSHW-Logo_5.7x6mm_SilkScreen, B.Cu at (103.8, 79.6)
- added REF**: KiCad-Logo2_5mm_SilkScreen, Symbol:KiCad-Logo2_5mm_SilkScreen, B.Cu at (103.6, 87.1)
- moved TP_3 3.88 mm to (113.6, 64.4)
- moved TP_GND1 3.12 mm to (106.1, 60.8)
- moved J7 2.70 mm to (199.9, 84.4)
- moved TH1 2.09 mm to (97.0, 59.8)
- moved R1 2.00 mm to (100.6, 62.2)
- moved C47 1.27 mm to (183.2, 72.9), turned to 180 degrees
- moved C45 1.25 mm to (183.0, 49.7), turned to 180 degrees
- moved C46 1.20 mm to (183.2, 62.5), turned to 180 degrees
- moved D1 1.06 mm to (112.9, 54.4)
- moved R2 0.84 mm to (108.9, 67.1)
- moved Q1 0.55 mm to (106.4, 67.4), turned to -90 degrees
- moved C31 0.46 mm to (148.7, 68.1)
- moved C28 0.42 mm to (150.2, 68.1)
- moved R6 0.40 mm to (123.2, 54.4)
- moved L4 0.38 mm to (141.6, 57.7)
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- renumbered TP_2 to TP_12V1
Connections:
- U3 pad 10: (no net) -> GND
- U3 pad 11: (no net) -> GND
- U3 pad 12: (no net) -> GND
- U3 pad 13: (no net) -> GND
- U3 pad 14: (no net) -> GND
- U3 pad 15: (no net) -> GND
Routing:
- net GND: track 0.05 -> 17.8 mm, vias 23 -> 230
- net +3V3: track 191.2 -> 206.0 mm, vias 49 -> 50
- net +1V1: track 26.3 -> 31.7 mm
- net +5V: track 100.1 -> 103.1 mm
- net Net-(U3-SW): track 2.18 -> 0.00 mm
- net /MOTB_IN: track 17.2 -> 19.2 mm
- net /MOTC_IN: track 24.6 -> 26.5 mm
- net /MOTA_IN: track 25.1 -> 26.8 mm
- net Net-(C45-Pad1): track 0.00 -> 1.72 mm
- net /DRV_SDO: track 33.8 -> 32.1 mm
- net Net-(C46-Pad1): track 0.00 -> 1.65 mm
- net Net-(C47-Pad1): track 0.00 -> 1.62 mm
- net /GPIO29_ADC3: track 58.6 -> 60.2 mm
- net /RUN: track 46.9 -> 45.7 mm, vias 3 -> 2
- net /DRV_nFAULT: track 33.2 -> 34.3 mm
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- added copper zone on F.Cu, net Net-(U1-SW)
- added copper zone on F.Cu, net Net-(U3-SW)
Other:
- board text added: "+"
- board text added: "-"
- board text added: "BOOT"
- board text added: "DEBUG"
- board text added: "DOUGHTER-BOARD"
- board text added: "DRV8350S"
- board text added: "Design by: Syauqi Alias"
- board text added: "Design by: Syauqi Alias for Manufacturing Futures Lab, UCL"
- board text added: "HALL SENS"
- board text added: "I2C"
- board text added: "POWER IN (30V-80V)"
- board text added: "RP2350"
- board text added: "RUN"
- board text added: "TE-005-1a"
- board text added: "TEMP-PROBE"
- board text added: "TP 12V"
- board text added: "TP 3V3"
- board text added: "TP 5V"
- board text added: "TP GND"
